File: aniket.kicad_pcb (KiCad board)
At the start: 2 copper layers, 71.1 x 40.6 mm, 16 parts, among them IC1 TEA2025B, J1 Conn_01x04_Male, J2 Conn_01x02_Male, J3 Conn_01x02_Male, J4 Barrel_Jack_Switch

Commit message: 2 One layer 0.8mm
Parts:
- moved J1 2.80 mm to (101.9, 96.4)
Routing:
- net /gnd: track 0.00 -> 303.7 mm
- net +5V: track 14.7 -> 58.7 mm
- net /IN1: track 50.8 -> 48.1 mm
- net /IN2: track 52.0 -> 49.4 mm
- net Net-(C9-Pad2): track 11.6 -> 12.7 mm
- added copper zone on F.Cu, net /gnd
- removed copper zone on F.Cu, net +5V
- removed copper zone on B.Cu, net /gnd
